Commit message: [Task 2.33] Test and perform code review

File: urdf/shamazon_robot.xacro (robot description, xacro)
@@ -66,5 +66,5 @@
         <box size="0.6 0.01 0.02"/>
       </geometry>
-      <origin rpy="0 0 0" xyz="0 0 0"/>
+      <origin rpy="0 0 0" xyz="0 -0.35 0"/>
     </visual> -->
     <collision>
@@ -72,5 +72,5 @@
         <box size="0.6 0.01 0.02"/>
       </geometry>
-      <origin rpy="0 0 0" xyz="0 0 0"/>
+      <origin rpy="0 0 0" xyz="0 -0.35 0"/>
     </collision>
     <inertial>
@@ -170,5 +170,5 @@
     <child link="conveyor2"/>
     <axis xyz="0 1 0"/>
-    <limit effort="1000.0" lower="-0.4" upper="0.4" velocity="0.5"/>
+    <limit effort="1000.0" lower="0" upper="0.7" velocity="0.5"/>
     <origin xyz="0 0 0.25" rpy="0 0 0" />
   </joint>
@@ -225,5 +225,5 @@
       <wheelDiameter>0.3555</wheelDiameter>
       <robotBaseFrame>robot_footprint</robotBaseFrame>
-      <torque>100</torque>
+      <torque>50</torque>
       <topicName>cmd_vel</topicName>
       <broadcastTF>true</broadcastTF>
@@ -315,6 +315,6 @@
   <gazebo reference="front_left_wheel">
     <material>Gazebo/Grey</material>
-    <mu1>0.1</mu1>
-    <mu2>0.1</mu2>
+    <mu1>0.5</mu1>
+    <mu2>0.5</mu2>
     <selfCollide>true</selfCollide>
     <minDepth>0.003</minDepth>
@@ -322,6 +322,6 @@
   <gazebo reference="back_left_wheel">
     <material>Gazebo/Grey</material>
-    <mu1>0.1</mu1>
-    <mu2>0.1</mu2>
+    <mu1>0.5</mu1>
+    <mu2>0.5</mu2>
     <selfCollide>true</selfCollide>
     <minDepth>0.003</minDepth>
@@ -329,6 +329,6 @@
   <gazebo reference="back_right_wheel">
     <material>Gazebo/Grey</material>
-    <mu1>0.1</mu1>
-    <mu2>0.1</mu2>
+    <mu1>0.5</mu1>
+    <mu2>0.5</mu2>
     <selfCollide>true</selfCollide>
     <minDepth>0.003</minDepth>
@@ -336,6 +336,6 @@
   <gazebo reference="front_right_wheel">
     <material>Gazebo/Grey</material>
-    <mu1>0.1</mu1>
-    <mu2>0.1</mu2>
+    <mu1>0.5</mu1>
+    <mu2>0.5</mu2>
     <selfCollide>true</selfCollide>
     <minDepth>0.003</minDepth>
